File: array/mems_array.kicad_pcb (KiCad board)
At the start: 4 copper layers, 350 x 190 mm, 61 parts, among them U101 74AHC244, U102 743245, U103 741G04, U104 BEAGLEBONEBLACK, U201 SN74CTBLV3251, U301 SN74CTBLV3251, U401 SN74CTBLV3251, U501 SN74CTBLV3251, U601 SN74CTBLV3251

Commit message: Fix PCB position in the page.
Signed-off-by: Chamon <luizchamon@gmail.com>
Parts:
- moved C101 53.2 mm to (285.1, 116.3)
- moved C102 53.2 mm to (287.0, 162.0)
- moved C501 53.2 mm to (145.2, 142.7)
- moved C601 53.2 mm to (145.4, 182.3)
- moved MIC201 53.2 mm to (65.0, 60.0)
- moved MIC202 53.2 mm to (76.0, 60.0)
- moved MIC203 53.2 mm to (98.0, 60.0)
- moved MIC204 53.2 mm to (131.0, 60.0)
- moved MIC205 53.2 mm to (153.0, 60.0)
- moved MIC206 53.2 mm to (197.0, 60.0)
- moved MIC207 53.2 mm to (241.0, 60.0)
- moved MIC208 53.2 mm to (263.0, 60.0)
- moved MIC301 53.2 mm to (65.0, 80.0)
- moved MIC302 53.2 mm to (76.0, 80.0)
- moved MIC303 53.2 mm to (98.0, 80.0)
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